Commit message: feat: Grounding DINO object detection + 3D PCA grasp angle + pick sequence
- object_tracking_node: zero-shot object detection via Grounding DINO,
  depth-based 3D positioning, 3D PCA grasp angle estimation,
  lock/unlock selection, obstacle publishing to cuRobo
- curobo_planner_node: pick sequence (open→descend→close→lift),
  dynamic obstacle update from detected objects, collision cache fix,
  MoveLine + Trigger service integration
- curobo_vision.launch.py: sequential launch (cuRobo first, then DINO),
  Grounding DINO as default mode
- marker_tracking_node: added pick support and angle adjustment
- E0509 joint limits corrected to actual robot spec
- README: complete rewrite of cuRobo vision section

Co-Authored-By: Claude Opus 4.6 (1M context) <noreply@anthropic.com>

File: config/curobo/e0509_gripper.urdf (robot description, URDF)
Before this commit: robot e0509_with_gripper, 13 links, 12 joints
Joints:
- joint joint_1: limit lower=-6.2832 upper=6.2832 effort=194 velocity=3.1416 -> lower=-6.283185307179586 upper=6.283185307179586 effort=194 velocity=3.1416
- joint joint_2: limit lower=-6.2832 upper=6.2832 effort=194 velocity=3.1416 -> lower=-1.6580627893946132 upper=1.6580627893946132 effort=194 velocity=3.1416
- joint joint_3: limit lower=-2.7053 upper=2.7053 effort=194 velocity=3.1416 -> lower=-2.356194490192345 upper=2.356194490192345 effort=194 velocity=3.1416
- joint joint_4: limit lower=-6.2832 upper=6.2832 effort=66 velocity=3.927 -> lower=-6.283185307179586 upper=6.283185307179586 effort=66 velocity=3.927
- joint joint_5: limit lower=-6.2832 upper=6.2832 effort=66 velocity=3.927 -> lower=-2.356194490192345 upper=2.356194490192345 effort=66 velocity=3.927
- joint joint_6: limit lower=-6.2832 upper=6.2832 effort=66 velocity=3.927 -> lower=-6.283185307179586 upper=6.283185307179586 effort=66 velocity=3.927
