Commit message: feat: organize strawberry harvest mini-project portfolio

File: config/curobo/e0509_gripper.urdf (robot description, URDF)
Before this commit: robot e0509_with_gripper, 13 links, 12 joints
Joints:
- joint joint_3: limit lower=-2.356194490192345 upper=2.356194490192345 effort=194 velocity=3.1416 -> lower=-2.7053 upper=2.7053 effort=194 velocity=3.1416

Commit message: feat: add measured grasp TCP validation workflow

File: config/curobo/e0509_gripper.urdf (robot description, URDF)
Before this commit: robot e0509_with_gripper, 13 links, 12 joints
Links:
- added link grasp_tcp_link
Joints:
- added joint grasp_tcp_joint: type fixed, parent gripper_rh_p12_rn_base, child grasp_tcp_link, origin xyz=0 0 0.260 rpy=0 0 0

File: urdf/e0509_with_gripper.urdf.xacro (robot description, xacro)
@@ -37,4 +37,11 @@
     <parent link="link_6"/>
     <child link="gripper_rh_p12_rn_base"/>
+  </joint>
+  <!-- Measured effective grasp center: 10mm behind the 270mm part tips. -->
+  <link name="grasp_tcp_link"/>
+  <joint name="grasp_tcp_joint" type="fixed">
+    <origin xyz="0 0 0.260" rpy="0 0 0"/>
+    <parent link="gripper_rh_p12_rn_base"/>
+    <child link="grasp_tcp_link"/>
   </joint>
   <!-- Gazebo ros2_control -->

Commit message: feat: validate continuous row2 tray descent

File: config/curobo/e0509_gripper.urdf (robot description, URDF)
Before this commit: robot e0509_with_gripper, 14 links, 13 joints
Joints:
- joint joint_3: limit lower=-2.7053 upper=2.7053 effort=194 velocity=3.1416 -> lower=-2.356194 upper=2.356194 effort=194 velocity=3.1416
